Commit message: feat(pybullet_magic_bin): add new environment with magic bin and block vanishing logic

File: predicators/envs/assets/urdf/partnet_mobility/bucket/100470/bucket.urdf (robot description, URDF)
Before this commit: robot partnet_af5f4299084775cb4bb0a929135b1b1f, 3 links, 2 joints
Links:
- removed link link_0
- link link_1: geometry collision box size=0.1 1.2 0.8; collision box size=0.1 1.2 0.8
Joints:
- removed joint joint_0

Commit message: fix(bucket): adjust collision dimensions and origins for walls

File: predicators/envs/assets/urdf/partnet_mobility/bucket/100470/bucket.urdf (robot description, URDF)
Before this commit: robot partnet_af5f4299084775cb4bb0a929135b1b1f, 2 links, 1 joints
Links:
- link link_1: geometry collision box size=0.1 0.8 0.8; collision box size=0.1 0.8 0.8
